File: Hardware/Pre-Ignition x4/MX4B/Fuel-Ignition.sch (KiCad schematic (older format))
At the start: 39 parts, among them Q5 STP62NS04Z, Q6 STP62NS04Z, Q7 STP62NS04Z, Q8 STP62NS04Z, U1 TC4427, U2 TC4427

Commit message: Pre-Ignition x2 Initial Upload, MX4B Production.
Pre-Ignition x2 Initial Upload - 2 Channel Speeduino compatible ECU
Pre-Ignition x4 MX4B (revision B) - minor updates, BOM changes, connectors moved to bottom side of board.
Parts:
- LED1, LED2, LED3, LED4: LCSC C2286 -> C72041
Changed lines of the file:
@@
 encoding utf-8
 Sheet 3 5
-Title ""
+Title "Pre-Ignition X4"
 Date ""
-Rev "1"
-Comp ""
-Comment1 ""
+Rev "2"
+Comp "DetonationEMS"
+Comment1 "detonationems.com"
 Comment2 ""
 Comment3 ""
@@
 F 3 "~" H 8850 1700 50  0001 C CNN
 F 4 "C2286" H 8850 1700 50  0001 C CNN "JLC"
-F 5 "C2286" H 8850 1700 50  0001 C CNN "LCSC"
+F 5 "C72041" H 8850 1700 50  0001 C CNN "LCSC"
 	1    8850 1700
 	-1   0    0    1
@@
 F 3 "~" H 8850 3200 50  0001 C CNN
 F 4 "C2286" H 8850 3200 50  0001 C CNN "JLC"
-F 5 "C2286" H 8850 3200 50  0001 C CNN "LCSC"
+F 5 "C72041" H 8850 3200 50  0001 C CNN "LCSC"
 	1    8850 3200
 	-1   0    0    1
@@
 F 3 "~" H 4000 1650 50  0001 C CNN
 F 4 "C2286" H 4000 1650 50  0001 C CNN "JLC"
-F 5 "C2286" H 4000 1650 50  0001 C CNN "LCSC"
+F 5 "C72041" H 4000 1650 50  0001 C CNN "LCSC"
 	1    4000 1650
 	-1   0    0    1
@@
 F 3 "~" H 4000 3150 50  0001 C CNN
 F 4 "C2286" H 4000 3150 50  0001 C CNN "JLC"
-F 5 "C2286" H 4000 3150 50  0001 C CNN "LCSC"
+F 5 "C72041" H 4000 3150 50  0001 C CNN "LCSC"
 	1    4000 3150
 	-1   0    0    1
