File: Hardware/Pre-Ignition x4/MX4B/Pre_Ignition.sch (KiCad schematic (older format))
At the start: 18 parts, among them IC1 L7805CDT

Commit message: Pre-Ignition x2 Initial Upload, MX4B Production.
Pre-Ignition x2 Initial Upload - 2 Channel Speeduino compatible ECU
Pre-Ignition x4 MX4B (revision B) - minor updates, BOM changes, connectors moved to bottom side of board.
Parts:
- D6, D7: LCSC C2286 -> C72043
Changed lines of the file:
@@
 Sheet 1 5
 Title "Pre-Ignition X4"
-Date "2021-08-11"
+Date "2021-09-21"
 Rev "2"
 Comp "DetonationEMS"
@@
 F 2 "LED_SMD:LED_0603_1608Metric" H 7450 4300 50  0001 C CNN
 F 3 "~" H 7450 4300 50  0001 C CNN
-F 4 "C2286" H 7450 4300 50  0001 C CNN "LCSC"
+F 4 "C72043" H 7450 4300 50  0001 C CNN "LCSC"
 	1    7450 4300
 	-1   0    0    1
@@
 F 2 "LED_SMD:LED_0603_1608Metric" H 7450 4550 50  0001 C CNN
 F 3 "~" H 7450 4550 50  0001 C CNN
-F 4 "C2286" H 7450 4550 50  0001 C CNN "LCSC"
+F 4 "C72043" H 7450 4550 50  0001 C CNN "LCSC"
 	1    7450 4550
 	-1   0    0    1
