File: Hardware/v1.3/1.3e/1.3.kicad_pcb (KiCad board)
At the start: 2 copper layers, 100 x 100 mm, 157 parts, among them IC1 L7805CDT, J1 Conn_02x20_Counter_Clockwise, J10 Conn_01x02, J11 Conn_01x02, J2 Conn_01x04, J3 Conn_02x16_Counter_Clockwise, J4 VR_Header, J5 Conn_01x02, J6 Conn_01x02, J7 Conn_02x16_Counter_Clockwise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

Commit message: bom fix
Parts:
- R55, R63: value 470 -> 220
