File: Hardware/v1.3/1.3e/Analog.sch (KiCad schematic (older format))
At the start: 55 parts, among them J4 VR_Header, U3 SRV05-4-P-T7, U4 SRV05-4-P-T7, U5 SRV05-4-P-T7, U6 SRV05-4-P-T7

Commit message: bom fix
Parts:
- R55, R63: value 470 -> 220; LCSC C23179 -> C22962
Changed lines of the file:
@@
 P 2150 6950
 F 0 "R63" V 1943 6950 50  0000 C CNN
-F 1 "470" V 2034 6950 50  0000 C CNN
+F 1 "220" V 2034 6950 50  0000 C CNN
 F 2 "Resistor_SMD:R_0603_1608Metric" V 2080 6950 50  0001 C CNN
 F 3 "~" H 2150 6950 50  0001 C CNN
 F 4 "" H 2150 6950 50  0001 C CNN "JLC"
-F 5 "C23179" H 2150 6950 50  0001 C CNN "LCSC"
+F 5 "C22962" H 2150 6950 50  0001 C CNN "LCSC"
 	1    2150 6950
 	0    -1   -1   0
@@
 P 2150 5850
 F 0 "R55" V 1943 5850 50  0000 C CNN
-F 1 "470" V 2034 5850 50  0000 C CNN
+F 1 "220" V 2034 5850 50  0000 C CNN
 F 2 "Resistor_SMD:R_0603_1608Metric" V 2080 5850 50  0001 C CNN
 F 3 "~" H 2150 5850 50  0001 C CNN
-F 4 "" H 2150 5850 50  0001 C CNN "JLC"
-F 5 "C23179" H 2150 5850 50  0001 C CNN "LCSC"
+F 4 "C22962" H 2150 5850 50  0001 C CNN "LCSC"
 	1    2150 5850
 	0    1    1    0
