File: Hardware/VR Conditioner NCV1124/RevA/Duel VR.sch (KiCad schematic (older format))
At the start: 17 parts, among them IC1 NCV1124, J1 Speedy VR Mount

Commit message: VR Conditioner Update
Update Schematic
Include Instructions
Update Readme
Parts:
- R1, R2, R3, R4: value 22k -> 16k; LCSC C17560 -> C17490
- R5: value 24k -> 18k; LCSC C23352 -> C25810
Changed lines of the file:
@@
 P 5600 3700
 F 0 "R2" V 5600 3650 50  0000 C CNN
-F 1 "22k" V 5500 3600 50  0000 C CNN
+F 1 "16k" V 5500 3600 50  0000 C CNN
 F 2 "Resistor_SMD:R_0805_2012Metric" V 5530 3700 50  0001 C CNN
 F 3 "~" H 5600 3700 50  0001 C CNN
-F 4 "C17560" V 5600 3700 50  0001 C CNN "LCSC"
+F 4 "C17490" V 5600 3700 50  0001 C CNN "LCSC"
 	1    5600 3700
 	0    1    1    0
@@
 P 5600 3450
 F 0 "R1" V 5600 3400 50  0000 C CNN
-F 1 "22k" V 5550 3250 50  0000 C CNN
+F 1 "16k" V 5550 3250 50  0000 C CNN
 F 2 "Resistor_SMD:R_0805_2012Metric" V 5530 3450 50  0001 C CNN
 F 3 "~" H 5600 3450 50  0001 C CNN
-F 4 "C17560" V 5600 3450 50  0001 C CNN "LCSC"
+F 4 "C17490" V 5600 3450 50  0001 C CNN "LCSC"
 	1    5600 3450
 	0    1    1    0
@@
 P 5600 3800
 F 0 "R3" V 5600 3750 50  0000 C CNN
-F 1 "22k" V 5700 3700 50  0000 C CNN
+F 1 "16k" V 5700 3700 50  0000 C CNN
 F 2 "Resistor_SMD:R_0805_2012Metric" V 5530 3800 50  0001 C CNN
 F 3 "~" H 5600 3800 50  0001 C CNN
-F 4 "C17560" V 5600 3800 50  0001 C CNN "LCSC"
+F 4 "C17490" V 5600 3800 50  0001 C CNN "LCSC"
 	1    5600 3800
 	0    1    1    0
@@
 P 5600 4000
 F 0 "R4" V 5600 3950 50  0000 C CNN
-F 1 "22k" V 5650 3800 50  0000 C CNN
+F 1 "16k" V 5650 3800 50  0000 C CNN
 F 2 "Resistor_SMD:R_0805_2012Metric" V 5530 4000 50  0001 C CNN
 F 3 "~" H 5600 4000 50  0001 C CNN
-F 4 "C17560" V 5600 4000 50  0001 C CNN "LCSC"
+F 4 "C17490" V 5600 4000 50  0001 C CNN "LCSC"
 	1    5600 4000
 	0    1    1    0
@@
 P 5850 4550
 F 0 "R5" V 5850 4500 50  0000 C CNN
-F 1 "24k" V 5950 4600 50  0000 C CNN
+F 1 "18k" V 5950 4600 50  0000 C CNN
 F 2 "Resistor_SMD:R_0603_1608Metric" V 5780 4550 50  0001 C CNN
 F 3 "~" H 5850 4550 50  0001 C CNN
-F 4 "C23352" V 5850 4550 50  0001 C CNN "LCSC"
+F 4 "C25810" V 5850 4550 50  0001 C CNN "LCSC"
 	1    5850 4550
 	-1   0    0    1
