File: Hardware/DetoSim4/Simulator.kicad_pcb (KiCad board)
At the start: 2 copper layers, 97.6 x 70 mm, 45 parts, among them J1 Conn_01x03, J2 Conn_02x20_Counter_Clockwise, J6 Header, J8 Conn_01x03

Commit message: DetoStim Upload
Product read upload
Connections:
- A1 pad 1: (no net) -> unconnected-(A1-Pad1)
- A1 pad 10: (no net) -> unconnected-(A1-Pad10)
- A1 pad 13: (no net) -> unconnected-(A1-Pad13)
- A1 pad 14: (no net) -> unconnected-(A1-Pad14)
- A1 pad 15: (no net) -> unconnected-(A1-Pad15)
- A1 pad 16: (no net) -> unconnected-(A1-Pad16)
- A1 pad 17: (no net) -> unconnected-(A1-Pad17)
- A1 pad 18: (no net) -> unconnected-(A1-Pad18)
- A1 pad 2: (no net) -> MC-D0
- A1 pad 20: (no net) -> unconnected-(A1-Pad20)
- A1 pad 21: (no net) -> unconnected-(A1-Pad21)
- A1 pad 22: (no net) -> unconnected-(A1-Pad22)
- A1 pad 23: (no net) -> unconnected-(A1-Pad23)
- A1 pad 24: (no net) -> unconnected-(A1-Pad24)
- A1 pad 25: (no net) -> unconnected-(A1-Pad25)
- A1 pad 26: (no net) -> unconnected-(A1-Pad26)
- A1 pad 28: (no net) -> unconnected-(A1-Pad28)
- A1 pad 3: (no net) -> unconnected-(A1-Pad3)
- A1 pad 30: (no net) -> unconnected-(A1-Pad30)
- A1 pad 5: (no net) -> unconnected-(A1-Pad5)
- A1 pad 6: (no net) -> unconnected-(A1-Pad6)
- A1 pad 7: (no net) -> unconnected-(A1-Pad7)
- A1 pad 8: (no net) -> unconnected-(A1-Pad8)
- A1 pad 9: (no net) -> unconnected-(A1-Pad9)
- J2 pad 14: (no net) -> FLEX
- J2 pad 15: (no net) -> FAN
- J2 pad 16: (no net) -> FP
- J2 pad 17: (no net) -> TACH
- J2 pad 18: (no net) -> CLUTCH
- J2 pad 26: (no net) -> VR2-
- J2 pad 27: (no net) -> VR1-
- J2 pad 29: (no net) -> 2B
- J2 pad 30: (no net) -> 2A
- J2 pad 31: (no net) -> 1A
- J2 pad 32: (no net) -> 1B
- J2 pad 35: (no net) -> BOOST
- J2 pad 36: (no net) -> IDLE2
- J2 pad 37: (no net) -> IDLE
- J2 pad 38: (no net) -> VVT
Other:
- net class Default removed
