File: Hardware/Engine Simulation/8 Channel/Simulator.kicad_sch (KiCad schematic)
At the start: 78 parts, among them J1 Conn_01x03, J10 Conn_01x04, J11 Conn_01x03, J2 Conn_02x20_Counter_Clockwise, J3 Conn_01x08, J4 Conn_01x04, J5 Conn_01x10, J6 Crank Trigger Voltage, J7 Cam Trigger Voltage, J8 Conn_01x08, J9 Conn_01x04, Q1 AO3400A, Q2 AO3400A, SW1 Switch

Commit message: Minor Corrections
Silkscreen Correction - Cam and Crank output labels were swapped

Output pulse LED's removed (Serve no purpose)

Minor layout improvements.
Parts:
- removed D2: SS34, Diode_SMD:D_SMA, symbol Device:D
- removed LED21: Crank Pulse, LED_SMD:LED_0603_1608Metric, symbol Device:LED
- removed LED22: Cam Pulse, LED_SMD:LED_0603_1608Metric, symbol Device:LED
- removed R29, R30: 470, Resistor_SMD:R_0603_1608Metric, symbol Device:R
- D1: footprint Diode_SMD:D_SMA -> Diode_SMD:D_SOD-123; LCSC C2480 -> C8598
- POT1, POT2, POT5, POT6: symbol Device:R_POT -> Detonation:Pot-10k; now in the parts list
- POT3: renamed from POT4; symbol Device:R_POT -> Detonation:Pot-10k; now in the parts list
- POT4: renamed from POT3; symbol Device:R_POT -> Detonation:Pot-10k; now in the parts list
- renumbered G3 to G2, G4 to G3, J2 to J1, J6 to J10, J7 to J11, J8 to J2, J10 to J4, J9 to J5, J4 to J6, J5 to J7, J1 to J8, J11 to J9, R3 to R1, R12 to R10, R13 to R11, R14 to R12, R15 to R13, R16 to R14, R17 to R15, R18 to R16, R19 to R17, R20 to R18, R22 to R19, R4 to R2, R21 to R20, R1 to R21, R2 to R22, R25 to R23, R23 to R24, R27 to R25, R28 to R26, R26 to R27, R24 to R28, R5 to R3, R6 to R4, R7 to R5, R8 to R6, R9 to R7, R10 to R8, R11 to R9
Connections:
- net +12V: now also A1.30 (VIN), D1.1 (K), J9.1 (Pin_1); no longer D1.2 (A), J10.1 (Pin_1), J11.1 (Pin_1), J6.1 (Pin_1)
- net +5V: now also J6.3 (Pin_3); no longer J6.2 (Pin_2)
- net CLT: now also J7.9 (Pin_9); no longer J7.7 (Pin_7)
- net GND: now also J6.2 (Pin_2), POT1.4 (Mounting_Tap), POT1.5 (Mounting_Tap), POT2.4 (Mounting_Tap), POT2.5 (Mounting_Tap), POT3.4 (Mounting_Tap), POT3.5 (Mounting_Tap), POT4.4 (Mounting_Tap), POT4.5 (Mounting_Tap), POT5.4 (Mounting_Tap), POT5.5 (Mounting_Tap), POT6.4 (Mounting_Tap), POT6.5 (Mounting_Tap); no longer J6.3 (Pin_3)
- net IAT: now also J7.10 (Pin_10); no longer J7.6 (Pin_6)
- net MAP: now also J7.6 (Pin_6); no longer J7.10 (Pin_10)
- net o2: now also J7.7 (Pin_7); no longer J7.9 (Pin_9)
- new net +BATT: D1.2 (A), J10.1 (Pin_1), J11.1 (Pin_1), J6.1 (Pin_1)
Other:
- moved on the sheet: D1, J6, J9, SW1
