File: Hardware/Modules/VR Conditioner NCV1124/RevA/Duel VR.kicad_sch (KiCad schematic)
At the start: 17 parts, among them IC1 NCV1124, J1 Speedy VR Mount

Commit message: Schematic Correction
VRConditioner NCV1124 schematic math correction.
Readme Updated for upcoming revision
Instructions Added to RevA folder
Parts:
- removed JP1, JP2: SolderJumper_2_Bridged, Jumper:SolderJumper-2_P1.3mm_Bridged_RoundedPad1.0x1.5mm, symbol Jumper:SolderJumper_2_Bridged
- removed R1, R4: 16k, Resistor_SMD:R_0805_2012Metric, symbol Device:R
Connections:
- net VR1OUT: now also IC1.7 (OUT1)
- net VR2OUT: now also IC1.6 (OUT2)
Other:
- note removed: "Cut Jumper if using hall sensor JP1 - CRANK JP2 - CAM"
- note removed: "R1+R2 1/2 Watt Min"
- note removed: "R3+R4 1/2 Watt Min"
Changed lines of the file:
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@@
     (comment 2 "github.com/DetonationEMS")
   )
-  (junction (at 137.16 93.98) (diameter 0) (color 0 0 0 0)
-  )
   (junction (at 146.05 96.52) (diameter 0) (color 0 0 0 0)
   )
-  (junction (at 137.16 96.52) (diameter 0) (color 0 0 0 0)
-  )
-  (junction (at 146.05 87.63) (diameter 0) (color 0 0 0 0)
-  )
   (junction (at 146.05 93.98) (diameter 0) (color 0 0 0 0)
   )
-  (junction (at 146.05 101.6) (diameter 0) (color 0 0 0 0)
-  )
   (junction (at 148.59 111.76) (diameter 0) (color 0 0 0 0)
   )
   (junction (at 182.88 87.63) (diameter 0) (color 0 0 0 0)
   )
+  (wire (pts (xy 182.88 99.06) (xy 190.5 99.06))
+    (stroke (width 0) (type default) (color 0 0 0 0))
+  )
   (wire (pts (xy 146.05 96.52) (xy 152.4 96.52))
     (stroke (width 0) (type default) (color 0 0 0 0))
   )
-  (wire (pts (xy 146.05 96.52) (xy 146.05 101.6))
+  (wire (pts (xy 182.88 96.52) (xy 190.5 96.52))
+    (stroke (width 0) (type default) (color 0 0 0 0))
+  )
+  (wire (pts (xy 146.05 96.52) (xy 146.05 107.95))
     (stroke (width 0) (type default) (color 0 0 0 0))
   )
@@
     (stroke (width 0) (type default) (color 0 0 0 0))
   )
-  (wire (pts (xy 137.16 101.6) (xy 138.43 101.6))
-    (stroke (width 0) (type default) (color 0 0 0 0))
-  )
   (wire (pts (xy 148.59 99.06) (xy 152.4 99.06))
     (stroke (width 0) (type default) (color 0 0 0 0))
   )
-  (wire (pts (xy 146.05 81.28) (xy 146.05 87.63))
-    (stroke (width 0) (type default) (color 0 0 0 0))
-  )
-  (wire (pts (xy 137.16 96.52) (xy 137.16 101.6))
-    (stroke (width 0) (type default) (color 0 0 0 0))
-  )
   (wire (pts (xy 182.88 87.63) (xy 182.88 81.28))
     (stroke (width 0) (type default) (color 0 0 0 0))
   )
-  (wire (pts (xy 138.43 87.63) (xy 137.16 87.63))
-    (stroke (width 0) (type default) (color 0 0 0 0))
-  )
-  (wire (pts (xy 137.16 87.63) (xy 137.16 93.98))
-    (stroke (width 0) (type default) (color 0 0 0 0))
-  )
-  (wire (pts (xy 146.05 87.63) (xy 146.05 93.98))
-    (stroke (width 0) (type default) (color 0 0 0 0))
-  )
-  (wire (pts (xy 146.05 101.6) (xy 146.05 107.95))
-    (stroke (width 0) (type default) (color 0 0 0 0))
-  )
-  (wire (pts (xy 137.16 93.98) (xy 138.43 93.98))
+  (wire (pts (xy 146.05 81.28) (xy 146.05 93.98))
+    (stroke (width 0) (type default) (color 0 0 0 0))
+  )
+  (wire (pts (xy 134.62 93.98) (xy 138.43 93.98))
     (stroke (width 0) (type default) (color 0 0 0 0))
   )
@@
     (stroke (width 0) (type default) (color 0 0 0 0))
   )
-  (wire (pts (xy 137.16 96.52) (xy 138.43 96.52))
-    (stroke (width 0) (type default) (color 0 0 0 0))
-  )
-  (wire (pts (xy 137.16 93.98) (xy 134.62 93.98))
-    (stroke (width 0) (type default) (color 0 0 0 0))
-  )
-  (wire (pts (xy 134.62 96.52) (xy 137.16 96.52))
+  (wire (pts (xy 134.62 96.52) (xy 138.43 96.52))
     (stroke (width 0) (type default) (color 0 0 0 0))
   )
@@
     (effects (font (size 1.27 1.27)) (justify left bottom))
   )
-  (text "Cut Jumper if using hall sensor\nJP1 - CRANK\nJP2 - CAM"
-    (at 186.69 109.22 0)
-    (effects (font (size 1.27 1.27)) (justify left bottom))
-  )
   (text "Speedy Compatible Mount" (at 86.36 115.57 0)
-    (effects (font (size 1.27 1.27)) (justify left bottom))
-  )
-  (text "R1+R2 \n1/2 Watt Min" (at 121.92 91.44 0)
-    (effects (font (size 1.27 1.27)) (justify left bottom))
-  )
-  (text "R3+R4\n1/2 Watt Min" (at 121.92 102.87 0)
     (effects (font (size 1.27 1.27)) (justify left bottom))
   )
@@
     (pin "2")
   )
-  (symbol (lib_id "Device:R") (at 142.24 87.63 270) (unit 1)
-    (in_bom yes) (on_board yes)
-    (property "Reference" "R1" (id 0) (at 140.97 87.63 90))
-    (property "Value" "16k" (id 1) (at 137.16 86.36 90))
-    (property "Footprint" "Resistor_SMD:R_0805_2012Metric" (id 2) (at 142.24 85.852 90)
-      (effects (font (size 1.27 1.27)) hide)
-    )
-    (property "Datasheet" "~" (id 3) (at 142.24 87.63 0)
-      (effects (font (size 1.27 1.27)) hide)
-    )
-    (property "LCSC" "C17490" (id 4) (at 142.24 87.63 90)
-      (effects (font (size 1.27 1.27)) hide)
-    )
-    (pin "1")
-    (pin "2")
-  )
   (symbol (lib_id "Device:R") (at 142.24 96.52 270) (unit 1)
     (in_bom yes) (on_board yes)
@@
     (pin "2")
   )
-  (symbol (lib_id "Device:R") (at 142.24 101.6 270) (unit 1)
-    (in_bom yes) (on_board yes)
-    (property "Reference" "R4" (id 0) (at 140.97 101.6 90))
-    (property "Value" "16k" (id 1) (at 137.16 102.87 90))
-    (property "Footprint" "Resistor_SMD:R_0805_2012Metric" (id 2) (at 142.24 99.822 90)
-      (effects (font (size 1.27 1.27)) hide)
-    )
-    (property "Datasheet" "~" (id 3) (at 142.24 101.6 0)
-      (effects (font (size 1.27 1.27)) hide)
-    )
-    (property "LCSC" "C17490" (id 4) (at 142.24 101.6 90)
-      (effects (font (size 1.27 1.27)) hide)
-    )
-    (pin "1")
-    (pin "2")
-  )
   (symbol (lib_id "Device:C") (at 142.24 81.28 90) (unit 1)
     (in_bom yes) (on_board yes)
@@
     )
   )
-  (symbol (lib_id "Jumper:SolderJumper_2_Bridged") (at 186.69 96.52 0) (unit 1)
-    (in_bom yes) (on_board yes)
-    (property "Reference" "JP1" (id 0) (at 186.69 93.6498 0))
-    (property "Value" "SolderJumper_2_Bridged" (id 1) (at 186.69 93.6244 0)
-      (effects (font (size 1.27 1.27)) hide)
-    )
-    (property "Footprint" "Jumper:SolderJumper-2_P1.3mm_Bridged_RoundedPad1.0x1.5mm" (id 2) (at 186.69 96.52 0)
-      (effects (font (size 1.27 1.27)) hide)
-    )
-    (property "Datasheet" "~" (id 3) (at 186.69 96.52 0)
-      (effects (font (size 1.27 1.27)) hide)
-    )
-    (pin "1")
-    (pin "2")
-  )
-  (symbol (lib_id "Jumper:SolderJumper_2_Bridged") (at 186.69 99.06 0) (unit 1)
-    (in_bom yes) (on_board yes)
-    (property "Reference" "JP2" (id 0) (at 186.69 101.6 0))
-    (property "Value" "SolderJumper_2_Bridged" (id 1) (at 186.69 96.1644 0)
-      (effects (font (size 1.27 1.27)) hide)
-    )
-    (property "Footprint" "Jumper:SolderJumper-2_P1.3mm_Bridged_RoundedPad1.0x1.5mm" (id 2) (at 186.69 99.06 0)
-      (effects (font (size 1.27 1.27)) hide)
-    )
-    (property "Datasheet" "~" (id 3) (at 186.69 99.06 0)
-      (effects (font (size 1.27 1.27)) hide)
-    )
-    (pin "1")
-    (pin "2")
-  )
   (sheet_instances
     (path "/" (page "1"))
@@
       (reference "J1") (unit 1) (value "Speedy VR Mount") (footprint "Misc:DIP-8_W7.62mm_Socket_VRConditioner")
     )
-    (path "/00000000-0000-0000-0000-00006158cac2"
-      (reference "JP1") (unit 1) (value "SolderJumper_2_Bridged") (footprint "Jumper:SolderJumper-2_P1.3mm_Bridged_RoundedPad1.0x1.5mm")
-    )
-    (path "/00000000-0000-0000-0000-00006158da3a"
-      (reference "JP2") (unit 1) (value "SolderJumper_2_Bridged") (footprint "Jumper:SolderJumper-2_P1.3mm_Bridged_RoundedPad1.0x1.5mm")
-    )
-    (path "/00000000-0000-0000-0000-0000612714d2"
-      (reference "R1") (unit 1) (value "16k") (footprint "Resistor_SMD:R_0805_2012Metric")
-    )
     (path "/00000000-0000-0000-0000-000061270210"
       (reference "R2") (unit 1) (value "16k") (footprint "Resistor_SMD:R_0805_2012Metric")
@@
       (reference "R3") (unit 1) (value "16k") (footprint "Resistor_SMD:R_0805_2012Metric")
     )
-    (path "/00000000-0000-0000-0000-000061272cf7"
-      (reference "R4") (unit 1) (value "16k") (footprint "Resistor_SMD:R_0805_2012Metric")
-    )
     (path "/00000000-0000-0000-0000-00006127bd11"
