File: Hardware/Engine Simulation/8 Channel/RevB/input.kicad_sch (KiCad schematic)
At the start: 58 parts, among them IC1 EL357NB_TA_-G, IC2 EL357NB_TA_-G, J1 Conn_02x20_Counter_Clockwise, J10 CMP PU, J11 CKP PU, J2 Conn_01x04, J3 Conn_01x08, J4 Conn_01x10

Commit message: Structure Update
MX2 - RevB Upload
MX4B-2 - KiCad Version update (no changes)
MX4C - Organized Schematic, Minor layout change
Engine Simulator 8 Channel - Organized Schematic (no changes)
PMAP-M - Map Sensor Breakout for MX4C
Other:
- company: (none) -> DetonationEMS
- title: (none) -> Engine Simulator
Changed lines of the file:
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@@
 (kicad_sch (version 20230121) (generator eeschema)
   (paper "A4")
+  (title_block
+    (title "Engine Simulator")
+    (date "2023-06-15")
+    (rev "Production B")
+    (company "DetonationEMS")
+  )
   (junction (at 34.29 74.93) (diameter 0) (color 0 0 0 0)
   )
