File: Hardware/Engine Simulation/8 Channel/RevB/simulation.kicad_sch (KiCad schematic)
At the start: 15 parts, among them J7 Conn_01x03, J8 Conn_01x03, SW1 Switch

Commit message: Structure Update
MX2 - RevB Upload
MX4B-2 - KiCad Version update (no changes)
MX4C - Organized Schematic, Minor layout change
Engine Simulator 8 Channel - Organized Schematic (no changes)
PMAP-M - Map Sensor Breakout for MX4C
Other:
- company: (none) -> DetonationEMS
- title: (none) -> Engine Simulator
Changed lines of the file:
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@@
 (kicad_sch (version 20230121) (generator eeschema)
   (paper "A4")
+  (title_block
+    (title "Engine Simulator")
+    (date "2023-06-15")
+    (rev "Production B")
+    (company "DetonationEMS")
+  )
   (junction (at 85.09 81.28) (diameter 0) (color 0 0 0 0)
   )
