File: Hardware/Engine Managment/Pre-Ignition/Pre-Ignition x4/End Cap/front/endcap.kicad_pcb (KiCad board)
At the start: 2 copper layers, 102.9 x 30.4 mm, 5 parts

Commit message: Minor updates
PMAP-M correction
Endcap updates
readme updates
Other:
- board text added: "OpenLogicEFI"
- board text removed: "DetonationEMS"
- board text removed: "JLCJLCJLCJLC"
