File: Hardware/Engine Managment/Closed Deck/Closed Deck x4/powersupply.kicad_sch (KiCad schematic)
At the start: 13 parts, among them IC1 7805

Commit message: schematic exports
kicad version updates, schematic exports
Parts:
- D1: LCSC C22452 -> C8678; Manufacture Part Number SS54 -> SS34
- D2: LCSC C3019524 -> C19077540; Manufacture Part Number P6SMAJ33CA -> SMAJ20CA
Other:
- note added: "SMAJ20CA"
- note removed: "SMAJ33CA"
Changed lines of the file:
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@@
 		)
 	)
-	(text "SMAJ33CA"
+	(text "SMAJ20CA"
 		(exclude_from_sim no)
 		(at 114.3 99.06 0)
@@
 			)
 		)
-		(property "LCSC" "C3019524"
+		(property "LCSC" "C19077540"
 			(at 119.38 92.71 90)
 			(effects
@@
 			)
 		)
-		(property "Manufacture Part Number" "P6SMAJ33CA"
+		(property "Manufacture Part Number" "SMAJ20CA"
 			(at 119.38 92.71 90)
 			(effects
@@
 			)
 		)
-		(property "LCSC" "C22452"
+		(property "LCSC" "C8678"
 			(at 125.73 88.9 0)
 			(effects
@@
 			)
 		)
-		(property "Manufacture Part Number" "SS54"
+		(property "Manufacture Part Number" "SS34"
 			(at 125.73 88.9 0)
 			(effects
