File: Hardware/Engine Managment/Pre-Ignition/Pre-Ignition x2/MX2B/Pre_Ignition.kicad_pcb (KiCad board)
At the start: 2 copper layers, 98.2 x 53.3 mm, 102 parts, among them IC1 L78M05ABDT-TR, IC2 MPXH6400, J1 VR_Header, J2 Conn_01x04, J3 Conn_01x04, J4 Conn_02x12_Counter_Clockwise, J5 Conn_01x04, J6 Conn_01x04, J7 Conn_01x04, Q1 STP62NS04Z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

Commit message: schematic exports
kicad version updates, schematic exports
Other:
- board text added: "A2 A1 B1 B2"
- board text removed: "locked"
