File: Hardware/Engine Managment/Pre-Ignition/Pre-Ignition x2/MX2B/Pre_Ignition.kicad_sch (KiCad schematic)
At the start: 0 parts

Commit message: schematic exports
kicad version updates, schematic exports
Other:
- removed sheet holdSheet
